Commit message: roboarm wheel twist issue solved

File: husky_description/urdf/wheel.urdf.xacro (robot description, xacro)
@@ -47,6 +47,4 @@
 			<kp value="10000000.0" />
 			<kd value="1.0" />
-			<fdir1 value="1 0 0"/>
-			<minDepth value="0.005" />
 		</gazebo>
 		<joint name="${wheel_prefix}_wheel" type="continuous">

File: roboarm/urdf/armbot/armbot.urdf.xacro (robot description, xacro)
@@ -1,10 +1,9 @@
 <?xml version="1.0"?>
-<robot name="roscontrol" xmlns:xacro="http://ros.org/wiki/xacro">
-  <xacro:property name="pi" value="3.1415" />
-  <xacro:property name="wheel_radius" value="0.15" />
-  <xacro:property name="wheel_thickness" value="0.1" />
-  <xacro:property name="chesis_length" value="0.6" />
-  <xacro:property name="chesis_breadth" value="0.4" />
-  <xacro:property name="chesis_height" value="0.2" />
+<robot name="armbot" xmlns:xacro="http://ros.org/wiki/xacro">
+  <xacro:property name="wheel_radius" value="0.08" />
+  <xacro:property name="wheel_thickness" value="0.04" />
+  <xacro:property name="chesis_length" value="0.3" />
+  <xacro:property name="chesis_breadth" value="0.2" />
+  <xacro:property name="chesis_height" value="0.08" />
   <material name="blue">
     <color rgba="0 0 0.8 1"/>
@@ -28,4 +27,5 @@
     </inertial>
   </xacro:macro>
+  <link name="base_link"></link>
   <link name="chesis">
     <visual>
@@ -40,6 +40,13 @@
       </geometry>
     </collision>
-    <xacro:box_inertia mass="10.0" x="${chesis_length}" y="${chesis_breadth}" z="${chesis_height}"/>
+    <xacro:box_inertia mass="0.5" x="${chesis_length}" y="${chesis_breadth}" z="${chesis_height}"/>
   </link>
+  <gazebo reference="chesis">
+       <material>Gazebo/Blue</material>
+    </gazebo>
+  <joint name="fixed_joint" type="fixed">
+      <parent link="base_link"/>
+      <child link="chesis"/>
+  </joint>
   <xacro:macro name="wheel" params="prefix suffix posx posy">
     <link name="${prefix}_${suffix}_wheel">
@@ -57,5 +64,5 @@
         </geometry>
       </collision>
-      <xacro:cyl_inertia mass="1" r="${wheel_radius}" h="${wheel_thickness}"/>
+      <xacro:cyl_inertia mass="0.1" r="${wheel_radius}" h="${wheel_thickness}"/>
     </link>
     <joint name="${prefix}_${suffix}_wheel_joint" type="continuous">
@@ -63,12 +70,9 @@
       <parent link="chesis"/>
       <child link="${prefix}_${suffix}_wheel"/>
-      <origin xyz="${0.25*posx} ${0.27*posy} 0" rpy="0 0 0"/>
+      <origin xyz="${(chesis_length*0.3)*posx} ${(chesis_breadth/2+wheel_thickness/2)*1.1*posy} 0" rpy="0 0 0"/>
+      <dynamics damping="0"/>
     </joint>
     <gazebo reference="${prefix}_${suffix}_wheel">
-      <mu1 value="200.0"/>
-      <mu2 value="100.0"/>
-      <kp value="10000000.0" />
-      <kd value="1.0" />
-      <material>Gazebo/Grey</material>
+       <material>Gazebo/DarkGray</material>
     </gazebo>
     <transmission name="${prefix}_${suffix}_wheel_trans">
@@ -86,8 +90,22 @@
   <xacro:wheel prefix="back" suffix="left" posx="-1" posy="1"/>
   <xacro:wheel prefix="back" suffix="right" posx="-1" posy="-1"/>
+  <xacro:include filename="$(find roboarm)/urdf/armbot/sensors.xacro"/>
+  <rgb_camera camera_name="armbot_rgb_camera" parent_link="chesis">
+    <box size="0.001 0.008 0.008"/>
+    <origin xyz="${(chesis_length/2)*1.001} 0 ${(chesis_height/2)*0.5}" rpy="0 0 0"/>
+  </rgb_camera>
+  <depth_camera camera_name="armbot_depth_camera" parent_link="chesis">
+    <box size="0.001 0.08 0.01"/>
+    <origin xyz="${(chesis_length/2)*1.001} 0 0" rpy="0 0 0"/>
+  </depth_camera>
+  <xacro:include filename="$(find roboarm)/urdf/turtlebot_arm/tbarm.xacro"/>
+  <turtlebot_arm parent="chesis" color="White" gripper_color="Green"
+                  pincher_gripper="false" turtlebot_gripper="true">
+    <origin xyz="0.1 0 0.06"/>
+  </turtlebot_arm>
   <!-- Gazebo plugin for ROS Control -->
   <gazebo>
     <plugin name="gazebo_ros_control" filename="libgazebo_ros_control.so">
-      <robotNamespace>/robot_base</robotNamespace>
+      <robotNamespace>/armbot</robotNamespace>
       <legacyModeNS>true</legacyModeNS>
       <robotSimType>gazebo_ros_control/DefaultRobotHWSim</robotSimType>

File: roboarm/urdf/armbot/sensors.xacro (robot description, xacro)
@@ -15,9 +15,9 @@
         </geometry>
       </visual>
-      <inertial>
+      <!-- <inertial>
         <mass value="0.01" />
         <origin xyz="0 0 0" rpy="0 0 0"/>
         <inertia ixx="5.3e-8" ixy="0" ixz="0" iyy="6.7e-9" iyz="0" izz="6.7e-9" />
-      </inertial>
+      </inertial> -->
     </link>
     <joint name="${camera_name}_joint" type="fixed">
@@ -50,5 +50,5 @@
           <alwaysOn>true</alwaysOn>
           <updateRate>0.0</updateRate>
-          <cameraName>roboarm/${camera_name}</cameraName>
+          <cameraName>armbot/${camera_name}</cameraName>
           <imageTopicName>image_raw</imageTopicName>
           <cameraInfoTopicName>camera_info</cameraInfoTopicName>
@@ -79,9 +79,9 @@
         </geometry>
       </visual>
-      <inertial>
+      <!-- <inertial>
         <mass value="0.05" />
         <origin xyz="0 0 0" rpy="0 0 0"/>
         <inertia ixx="2.7e-5" ixy="0" ixz="0" iyy="4.2e-7" iyz="0" izz="2.67e-5" />
-      </inertial>
+      </inertial> -->
     </link>
     <joint name="${camera_name}_joint" type="fixed">
@@ -167,5 +167,5 @@
         <topic>__default_topic__</topic>
         <plugin filename="libgazebo_ros_imu_sensor.so" name="imu_plugin">
-          <topicName>roboarm/${imu_name}</topicName>
+          <topicName>armbot/${imu_name}</topicName>
           <bodyName>${imu_name}_link</bodyName>
           <updateRateHZ>30.0</updateRateHZ>
