Commit message: Gripper working

File: roboarm/urdf/armbot/sensors.xacro (robot description, xacro)
@@ -50,5 +50,5 @@
           <alwaysOn>true</alwaysOn>
           <updateRate>0.0</updateRate>
-          <cameraName>armbot/${camera_name}</cameraName>
+          <cameraName>${camera_name}</cameraName>
           <imageTopicName>image_raw</imageTopicName>
           <cameraInfoTopicName>camera_info</cameraInfoTopicName>
@@ -91,45 +91,53 @@
       <child link="${camera_name}"/>
     </joint>
-  <gazebo reference="${camera_name}">
-    <sensor name="${camera_name}_camera" type="depth">
-      <update_rate>20</update_rate>
-      <camera>
-        <horizontal_fov>1.047198</horizontal_fov>
-        <image>
-          <width>640</width>
-          <height>480</height>
-          <format>R8G8B8</format>
-        </image>
-        <clip>
-          <near>0.05</near>
-          <far>3</far>
-        </clip>
-      </camera>
-      <plugin name="${camera_name}_controller" filename="libgazebo_ros_openni_kinect.so">
-        <baseline>0.2</baseline>
-        <alwaysOn>true</alwaysOn>
-        <updateRate>1.0</updateRate>
-        <cameraName>${camera_name}_ir</cameraName>
-        <imageTopicName>/${camera_name}/depth/image_raw</imageTopicName>
-        <cameraInfoTopicName>/${camera_name}/depth/camera_info</cameraInfoTopicName>
-        <depthImageTopicName>/${camera_name}/depth/image_raw</depthImageTopicName>
-        <depthImageInfoTopicName>/${camera_name}/depth/camera_info</depthImageInfoTopicName>
-        <pointCloudTopicName>/${camera_name}/depth/points</pointCloudTopicName>
-        <frameName>${camera_name}</frameName>
-        <pointCloudCutoff>0.5</pointCloudCutoff>
-        <pointCloudCutoffMax>3.0</pointCloudCutoffMax>
-        <distortionK1>0.00000001</distortionK1>
-        <distortionK2>0.00000001</distortionK2>
-        <distortionK3>0.00000001</distortionK3>
-        <distortionT1>0.00000001</distortionT1>
-        <distortionT2>0.00000001</distortionT2>
-        <CxPrime>0</CxPrime>
-        <Cx>0</Cx>
-        <Cy>0</Cy>
-        <focalLength>0</focalLength>
-        <hackBaseline>0</hackBaseline>
-      </plugin>
-    </sensor>
-  </gazebo>
+    <link name="camera_depth_link"></link>
+    <joint name="cameraLeft_depth_joint" type="fixed">
+      <origin xyz="0 0 0" rpy="-${pi/2} 0 -${pi/2} "/>
+      <parent link="${camera_name}"/>
+      <child link="camera_depth_link"/>
+    </joint>
+    <!-- Additional transformation link needed due to frame convention mismatch between gazebo and kinect in rviz
+    https://answers.ros.org/question/218395/libgazebo_ros_openni_kinectso-depth-pointcloud-wrong-tf/ -->
+    <gazebo reference="${camera_name}">
+      <sensor name="${camera_name}_camera" type="depth">
+        <update_rate>20</update_rate>
+        <camera>
+          <horizontal_fov>1.047198</horizontal_fov>
+          <image>
+            <width>640</width>
+            <height>480</height>
+            <format>R8G8B8</format>
+          </image>
+          <clip>
+            <near>0.001</near>
+            <far>3</far>
+          </clip>
+        </camera>
+        <plugin name="${camera_name}_controller" filename="libgazebo_ros_openni_kinect.so">
+          <baseline>0.2</baseline>
+          <alwaysOn>true</alwaysOn>
+          <updateRate>1.0</updateRate>
+          <cameraName>${camera_name}_ir</cameraName>
+          <imageTopicName>/${camera_name}/depth/image_raw</imageTopicName>
+          <cameraInfoTopicName>/${camera_name}/depth/camera_info</cameraInfoTopicName>
+          <depthImageTopicName>/${camera_name}/depth/image_raw</depthImageTopicName>
+          <depthImageInfoTopicName>/${camera_name}/depth/camera_info</depthImageInfoTopicName>
+          <pointCloudTopicName>/${camera_name}/depth/points</pointCloudTopicName>
+          <frameName>camera_depth_link</frameName>
+          <pointCloudCutoff>0.001</pointCloudCutoff>
+          <pointCloudCutoffMax>3.0</pointCloudCutoffMax>
+          <distortionK1>0.00000001</distortionK1>
+          <distortionK2>0.00000001</distortionK2>
+          <distortionK3>0.00000001</distortionK3>
+          <distortionT1>0.00000001</distortionT1>
+          <distortionT2>0.00000001</distortionT2>
+          <CxPrime>0</CxPrime>
+          <Cx>0</Cx>
+          <Cy>0</Cy>
+          <focalLength>0</focalLength>
+          <hackBaseline>0</hackBaseline>
+        </plugin>
+      </sensor>
+    </gazebo>
   </xacro:macro>
   <xacro:macro name="imu" params="imu_name parent_link *box *origin">

File: roboarm/urdf/turtlebot_arm/turtlebot_gripper.xacro (robot description, xacro)
@@ -49,3 +49,33 @@
       <origin xyz="0 0 0" rpy="0 0 ${M_PI}"/>
     </finger_fixed>
+    <gazebo reference="gripper_static_finger_link">
+			<mu1 value="100.0"/>
+			<mu2 value="50.0"/>
+			<kp value="10000000.0" />
+			<kd value="1.0" />
+		</gazebo>
+    <gazebo reference="gripper_active_finger_link">
+			<mu1 value="100.0"/>
+			<mu2 value="50.0"/>
+			<kp value="10000000.0" />
+			<kd value="1.0" />
+		</gazebo>
+    <gazebo>
+      <plugin name="gazebo_grasp_fix" filename="libgazebo_grasp_fix.so">
+        <robotNamespace>/armbot</robotNamespace>
+          <arm>
+            <arm_name>armbot</arm_name>
+            <gripper_link>gripper_active_link</gripper_link>
+            <gripper_link>arm_wrist_flex_link</gripper_link>
+            <palm_link>arm_wrist_flex_link</palm_link>
+          </arm>
+        <forces_angle_tolerance>100</forces_angle_tolerance>
+        <update_rate>4</update_rate>
+        <grip_count_threshold>4</grip_count_threshold>
+        <max_grip_count>8</max_grip_count>
+        <release_tolerance>0.005</release_tolerance>
+        <disable_collisions_on_attach>false</disable_collisions_on_attach>
+        <contact_topic>__default_topic__</contact_topic>
+      </plugin>
+    </gazebo>
 </robot>
